File: hardware/hackrf-one/baseband.sch (KiCad schematic (older format))
At the start: 136 parts, among them P14 XCVR_CLKOUT, P15 INTR, P16 CLKIN, P18 OEB, P2 CLKOUT, P36 VAA, P37 SCL, P38 SDA, P39 SSP1_SCK, P40 SSP1_MOSI, P41 SSP1_MISO, P53 CS_XCVR, P54 CS_AD, P55 TXENABLE, P56 RXENABLE, P57 XTAL2, P58 GCK1, P59 GCK2, P60 SGPIO_CLK, P61 DA0, P62 DA7, P63 DD0, P64 DD9, P65 DA4, P66 DD5, P67 RSSI, P83 GND, P84 GND, P85 GND, P86 GND, P87 GND, P88 GND, P89 GND, P9 BASEBAND, P90 GND, P91 GND, P92 GND, Q3 MOSFET_P, T3 RX_BALUN, T4 TX_BALUN, U17 MAX2837, U18 MAX5864, U19 SI5351C, X1 GSG-XTAL4PIN

Commit message: Corrected libraries (to use gsg-kicad-lib) and added SMP1330 protection
Parts:
- C100, C101, C102, C103, C104, C105, C106, C107, C108, C109, C110, C111, C112, C113, C114, C115, C116, C119, C120, C121, C122, C123, C124, C159, C165, C167, C168, C169, C170, C68, C69, C71, C72, C73, C74, C75, C76, C77, C78, C79, C80, C81, C82, C83, C84, C85, C86, C87, C88, C89, C90, C91, C92, C93, C94, C95, C96, C97, C98, C99: symbol C -> hackrf-one-rescue:C
- D3, D9: symbol GSG-DIODE-TVS-BI -> hackrf-one-rescue:GSG-DIODE-TVS-BI
- FB2: symbol FILTER -> hackrf-one-rescue:FILTER
- L6, L7, L8, L9: symbol INDUCTOR -> hackrf-one-rescue:INDUCTOR
- P14, P15, P18, P37, P38, P39, P40, P41, P53, P54, P55, P56, P57, P58, P59, P60, P61, P62, P63, P64, P65, P66, P67, P83, P84, P85, P86, P87, P88, P89, P90, P91, P92: symbol CONN_1 -> hackrf-one-rescue:CONN_1
- P16, P2: symbol GSG-RF-CONN -> hackrf-one-rescue:GSG-RF-CONN
- P36: symbol CONN_2 -> hackrf-one-rescue:CONN_2
- P9: symbol CONN_8X2 -> hackrf-one-rescue:CONN_8X2
- Q3: symbol MOSFET_P -> hackrf-one-rescue:MOSFET_P
- R10, R104, R105, R11, R13, R14, R15, R16, R17, R20, R21, R22, R23, R25, R26, R27, R28, R31, R32, R33, R41, R8, R85, R9, R94: symbol R -> hackrf-one-rescue:R
- T3, T4: symbol BALUN -> hackrf-one-rescue:BALUN
- U17: symbol MAX2837 -> hackrf-one-rescue:MAX2837
- U18: symbol MAX5864 -> hackrf-one-rescue:MAX5864
- U19: symbol SI5351C -> hackrf-one-rescue:SI5351C
- X1: symbol GSG-XTAL4PIN -> hackrf-one-rescue:GSG-XTAL4PIN
Connections:
- wire segments 320 -> 425
