File: hardware/hackrf-one/mcu.sch (KiCad schematic (older format))
At the start: 134 parts, among them J1 USB-MICRO-B, P1 1V8, P20 GPIO, P22 I2S, P23 DBGEN, P24 TRST, P25 LPC_ISP, P26 LPC_JTAG, P28 SD, P29 CPLD_JTAG, P3 GND, P30 BANK2_AUX, P5 LEDS, P68 SPIFI_CS, P69 VREGMODE, P70 EN_1V8, P71 ID, P72 GP_CLKIN, P73 P1_2, P74 P1_1, P75 GP_CLKIN, P76 GP_CLKIN, P77 GP_CLKIN, P78 GP_CLKIN, P79 GP_CLKIN, P8 VCC, P80 SHIELD, P81 SPIFI_SIO2, P82 SPIFI_SIO3, Q5 MOSFET_P, SW1 DFU, SW2 RESET, U15 TVS, U20 W25Q80, U21 TPS62410, U23 LPC4320FBD144, U24 GSG-XC2C64A-7VQG100C, X2 MCU_XTAL, X3 RTC_XTAL

Commit message: Corrected libraries (to use gsg-kicad-lib) and added SMP1330 protection
Parts:
- C118, C125, C126, C127, C128, C129, C130, C131, C132, C133, C134, C135, C136, C137, C138, C139, C140, C141, C142, C143, C144, C145, C146, C147, C148, C149, C150, C151, C152, C153, C154, C155, C156, C157, C158, C164: symbol C -> hackrf-one-rescue:C
- D2, D4, D5, D6, D7, D8: symbol LED -> hackrf-one-rescue:LED
- FB1, FB3: symbol FILTER -> hackrf-one-rescue:FILTER
- J1: symbol GSG-USB-MICRO-B-SHIELDED -> hackrf-one-rescue:GSG-USB-MICRO-B-SHIELDED
- L10, L11: symbol INDUCTOR -> hackrf-one-rescue:INDUCTOR
- P1, P29, P3, P8, P80: symbol CONN_2 -> hackrf-one-rescue:CONN_2
- P20, P28: symbol CONN_11X2 -> hackrf-one-rescue:CONN_11X2
- P22: symbol CONN_13X2 -> hackrf-one-rescue:CONN_13X2
- P23, P24, P68, P69, P70, P71, P72, P73, P74, P75, P76, P77, P78, P79, P81, P82: symbol CONN_1 -> hackrf-one-rescue:CONN_1
- P25: symbol CONN_6 -> hackrf-one-rescue:CONN_6
- P26: symbol CONN_5X2 -> hackrf-one-rescue:CONN_5X2
- P30: symbol CONN_10X2 -> hackrf-one-rescue:CONN_10X2
- P5: symbol CONN_3X2 -> hackrf-one-rescue:CONN_3X2
- Q5: symbol MOSFET_P -> hackrf-one-rescue:MOSFET_P
- R100, R12, R18, R19, R30, R34, R35, R37, R46, R47, R48, R49, R51, R52, R54, R55, R56, R57, R58, R59, R62, R63, R64, R65, R66, R67, R68, R69, R7, R72, R73, R74, R75, R76, R77, R78, R79, R80, R81, R86, R87, R88, R89, R90, R91, R93, R96, R98, R99: symbol R -> hackrf-one-rescue:R
- SW1, SW2: symbol SW_PUSH_SHIELDED -> hackrf-one-rescue:SW_PUSH_SHIELDED
- U15: symbol LXES1TBCC2-004 -> hackrf-one-rescue:LXES1TBCC2-004
- U20: symbol W25Q80BV -> hackrf-one-rescue:W25Q80BV
- U21: symbol TPS62410 -> hackrf-one-rescue:TPS62410
- U23: symbol LPC43XXFBD144 -> hackrf-one-rescue:LPC43XXFBD144
- U24: symbol GSG-XC2C64A-7VQG100C -> hackrf-one-rescue:GSG-XC2C64A-7VQG100C
- X2: symbol GSG-XTAL4PIN -> hackrf-one-rescue:GSG-XTAL4PIN
- X3: symbol CRYSTAL -> hackrf-one-rescue:CRYSTAL
